File: newproj/newproj.kicad_pcb (KiCad board)
At the start: 2 copper layers, 0 parts

Commit message: pcb layout draft
Parts:
- added C1: 10u/16v, Capacitor_SMD:CP_Elec_6.3x3.9, F.Cu at (77.3, 110.0)
- added C10: 100n, Capacitor_SMD:C_0603_1608Metric, F.Cu at (144.0, 70.0)
- added C11: 100n, Capacitor_SMD:C_0603_1608Metric, F.Cu at (146.0, 70.0)
- added C12: 100n, Capacitor_SMD:C_0603_1608Metric, F.Cu at (148.5, 70.0)
- added C13: 2u2/6v3, Capacitor_SMD:CP_Elec_4x3, F.Cu at (170.8, 125.8)
- added C14: 2u2/6v3, Capacitor_SMD:CP_Elec_4x3, F.Cu at (170.8, 131.6)
- added C15: 2u2/6v3, Capacitor_SMD:CP_Elec_4x3, F.Cu at (170.8, 137.4)
- added C16: 100n, Capacitor_SMD:C_0603_1608Metric, F.Cu at (170.0, 117.2)
- added C17: 100n, Capacitor_SMD:C_0603_1608Metric, F.Cu at (170.0, 119.8)
- added C18: 100n, Capacitor_SMD:C_0603_1608Metric, F.Cu at (102.2, 70.5)
- added C2: 10u/16v, Capacitor_SMD:CP_Elec_6.3x3.9, F.Cu at (77.0, 125.8)
- added C3: 10u/16v, Capacitor_SMD:CP_Elec_6.3x3.9, F.Cu at (77.0, 134.0)
- added C4: 100n, Capacitor_SMD:C_0603_1608Metric, F.Cu at (77.0, 139.5)
- added C5: 100n, Capacitor_SMD:C_0603_1608Metric, F.Cu at (77.0, 142.0)
- added C6: 100n, Capacitor_SMD:C_0603_1608Metric, F.Cu at (77.0, 144.5)
- added C7: 2u2/6v3, Capacitor_SMD:CP_Elec_4x3, F.Cu at (127.0, 70.0)
- added C8: 2u2/6v3, Capacitor_SMD:CP_Elec_4x3, F.Cu at (133.0, 70.2)
- added C9: 2u2/6v3, Capacitor_SMD:CP_Elec_4x3, F.Cu at (140.0, 70.0)
- added D1: 1N4002, Diode_SMD:D_SMA, F.Cu at (138.0, 117.0)
- added F1: 10A, Fuse:Fuseholder_Clip-5x20mm_Littelfuse_520_Inline_P20.50x5.80mm_D1.30mm_Horizontal, F.Cu at (174.2, 45.0)
- added F2: 10A, Fuse:Fuseholder_Clip-5x20mm_Littelfuse_520_Inline_P20.50x5.80mm_D1.30mm_Horizontal, F.Cu at (177.2, 71.0)
- added J1: AC CONN, TerminalBlock:TerminalBlock_bornier-2_P5.08mm, F.Cu at (74.0, 36.5)
- added J2: LED STRIP, Connector_Molex:Molex_Micro-Fit_3.0_43650-0315_1x03_P3.00mm_Vertical, F.Cu at (75.0, 117.6)
- added J3: SWD, Connector_PinHeader_2.54mm:PinHeader_1x04_P2.54mm_Vertical, F.Cu at (113.9, 70.0)
- added J4: Thermocouple, TerminalBlock:TerminalBlock_bornier-2_P5.08mm, F.Cu at (118.5, 147.0)
- added J5: HC MODULE, Connector_PinHeader_2.54mm:PinHeader_1x04_P2.54mm_Vertical, F.Cu at (165.0, 124.1)
- added J6: Higher Heater, TerminalBlock:TerminalBlock_bornier-2_P5.08mm, F.Cu at (184.4, 56.0)
- added J7: Lower Heater, TerminalBlock:TerminalBlock_bornier-2_P5.08mm, F.Cu at (184.4, 80.0)
- added J8: TOUCH DISPLAY, Connector_PinHeader_2.54mm:PinHeader_1x14_P2.54mm_Vertical, F.Cu at (107.0, 70.1)
- added J9: Electromagnet, TerminalBlock:TerminalBlock_bornier-2_P5.08mm, F.Cu at (136.5, 129.0)
- added PS1: IRM-10-3.3, Converter_ACDC:Converter_ACDC_MeanWell_IRM-10-xx_THT, F.Cu at (105.8, 51.5)
- added PS2: IRM-02-12, Converter_ACDC:Converter_ACDC_MeanWell_IRM-02-xx_THT, F.Cu at (205.5, 67.0)
- added PS3: IRM-20-5, Converter_ACDC:Converter_ACDC_MeanWell_IRM-20-xx_THT, F.Cu at (74.7, 95.8)
- added Q1: BT139-600, Package_TO_SOT_THT:TO-220-3_Vertical, F.Cu at (168.9, 57.9)
- added Q2: BT139-600, Package_TO_SOT_THT:TO-220-3_Vertical, F.Cu at (183.4, 100.0)
- added Q3: BS107, Package_TO_SOT_THT:TO-92_Inline, F.Cu at (123.7, 130.0)
- added R1: 220R, Resistor_SMD:R_0603_1608Metric, F.Cu at (167.4, 66.0)
- added R2: 220R, Resistor_SMD:R_0603_1608Metric, F.Cu at (167.4, 68.5)
- added R3: 220R, Resistor_SMD:R_0603_1608Metric, F.Cu at (167.4, 71.0)
- added R4: 220R, Resistor_SMD:R_0603_1608Metric, F.Cu at (175.4, 103.0)
- added R5: 220R, Resistor_SMD:R_0603_1608Metric, F.Cu at (175.4, 106.0)
- added R6: 220R, Resistor_SMD:R_0603_1608Metric, F.Cu at (171.4, 106.0)
- added R7: 10k, Resistor_SMD:R_0603_1608Metric, F.Cu at (165.0, 136.8)
- added R8: 10k, Resistor_SMD:R_0603_1608Metric, F.Cu at (124.0, 119.0)
- added SW1: PWR SWITCH, Connector_PinHeader_2.54mm:PinHeader_1x04_P2.54mm_Vertical, F.Cu at (86.4, 38.0)
- added SW2: PROJECT ~{RESET}, Button_Switch_SMD:SW_SPST_PTS645, F.Cu at (169.0, 145.0)
- added U1: MOC3041M, Package_DIP:DIP-6_W7.62mm, F.Cu at (155.7, 56.5)
- added U2: MOC3041M, Package_DIP:DIP-6_W7.62mm, F.Cu at (162.7, 92.5)
- added U3: ATSAML21G16B-AUT, Package_QFP:TQFP-48_7x7mm_P0.5mm, F.Cu at (120.0, 87.0)
Other:
- board outline added: 158 x 121 mm
- rule pad_to_mask_clearance: 0.05 -> 0
